File: docs/schematics/eagle/LeguinoNano.sch (EAGLE design)
At the start: 32 parts, among them Q1 60V/32A/35m?, Q2 60V/32A/35m?, Q3 60V/32A/35m?, Q4 60V/32A/35m?, Q5 60V/32A/35m?

Commit message: Continued EAGLE schematic and board for Arduino Uno.
Parts:
- removed NANO_L, NANO_R: (no value), pinhead:PINHD-1X15
- added JP1, JP2: (no value), pinhead:PINHD-1X8
- added JP3, JP4: (no value), pinhead:PINHD-1X6
- C1: device resistor:CPOL-USB -> adafruit:C-US050-030X075
Connections:
- removed net N$12: IN_2.3, IN_3.3, IN_4.3, IN_5.3, IN_6.3
- removed net NANO_3V3: NANO_R.14
- removed net NANO_5V: NANO_R.4
- removed net NANO_A0: NANO_R.12
- removed net NANO_A1: NANO_R.11
- removed net NANO_A2: IN_1.2, NANO_R.10
- removed net NANO_A3: IN_2.2, NANO_R.9
- removed net NANO_A4: IN_3.2, NANO_R.8
- removed net NANO_A5: IN_4.2, NANO_R.7
- removed net NANO_A6: IN_5.2, NANO_R.6
- removed net NANO_A7: IN_6.2, NANO_R.5
- removed net NANO_D0: NANO_L.1
- removed net NANO_D1: NANO_L.2
- removed net NANO_D10: NANO_L.13, Q4.G, R4.1
- removed net NANO_D11: NANO_L.14, Q5.G, R5.1
- removed net NANO_D12: NANO_L.15
- removed net NANO_D13: NANO_R.15
- removed net NANO_D2: NANO_L.5, REL1.5, REL2.5, REL3.5
- removed net NANO_D3: NANO_L.6, Q1.G, R1.1
- removed net NANO_D4: NANO_L.7, PLAY.2, Q2.G, R2.1
- removed net NANO_D5: NANO_L.8, Q3.G, R3.1
- removed net NANO_D6: NANO_L.9
- removed net NANO_D7: NANO_L.10, REL1.1
- removed net NANO_D8: NANO_L.11, REL3.1
- removed net NANO_D9: NANO_L.12, REL2.1
- removed net NANO_GND: NANO_L.4, NANO_R.2
- removed net NANO_REF: NANO_R.13
- removed net NANO_RST: NANO_L.3, NANO_R.3, RST.2
- removed net NANO_VIN: NANO_R.1
- new net UNO_A0: IN_1.2, JP4.1
- new net UNO_A1: IN_2.2, JP4.2
- new net UNO_A2: IN_3.2, JP4.3
- new net UNO_A3: IN_4.2, JP4.4
- new net UNO_A4: IN_5.2, JP4.5
- new net UNO_A5: IN_6.2, JP4.6
- new net UNO_D10: JP1.6, Q4.G, R4.1
- new net UNO_D11: JP1.5, Q5.G, R5.1
- new net UNO_D2: JP2.6, REL1.5, REL2.5, REL3.5
- new net UNO_D3: JP2.5, Q1.G, R1.1
- new net UNO_D4: JP2.4, PLAY.2
- new net UNO_D5: JP2.3, Q2.G, R2.1
- new net UNO_D6: JP2.2, Q3.G, R3.1
- new net UNO_D7: JP2.1, REL1.1
- new net UNO_D8: JP1.8, REL3.1
- new net UNO_D9: JP1.7, REL2.1
- new net UNO_RST: JP3.6, RST.2
- net GND: now also C1.2, JP1.2, JP3.2, JP3.3; no longer C1.-
- net V+: no longer IN_1.3
- net VCC: now also C1.1, IN_1.3, IN_2.3, IN_3.3, IN_4.3, IN_5.3, IN_6.3, JP3.1; no longer C1.+
Other:
- note removed: "Arduino Nano"
- moved on the sheet: D1, OUT_A, OUT_B, OUT_C, OUT_D, OUT_E, PLAY, PWR, Q4, Q5, R4, R5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
